File: test1/kicad/connectors.kicad_sch (KiCad schematic)
At the start: 0 parts

Commit message: test1: fill in Power, Bias, Bobcat, Connectors, FMC sheets
Completes the test1 Bobcat carrier hierarchical schematic. All 7 sheets
(root + 6 children) parse cleanly with kicad-cli and render to SVG/PDF.

Contents per child:
  - power.kicad_sch       — TPS7A8401A LDO (3P3V → 0.8V via ANY-OUT
                            strap, OUT side fans to +VDDD/+VDDA1/+VDDA2
                            via 1×2 jumpers) + TPS22916 load switch
                            (VADJ → +VDDIO) with EN pulldowns + decoupling.
  - bobcat.kicad_sch      — Bobcat 40-QFN DUT with VDDD/VDDIO decoupling,
                            VDDA1/VDDA2 series 0Ω + decoupling, hier-label
                            exits on all four edges for SAMPLE_OUT*,
                            SPI, GPIO, CLK_OUT*, BIAS0/1, etc.
  - eeprom.kicad_sch      — 24AA08 I²C EEPROM (address 000, WP→GND,
                            0.1 µF decoupling, 2.2 kΩ I²C pull-ups).
  - bias.kicad_sch        — MCP4728 quad DAC + OPA2388 dual op-amp
                            (units 1 & 2) + PMZ1200UPEYL high-side PMOS
                            × 2 channels + 5.11 kΩ 0.1% sense resistors +
                            DNP 2N7002 isolation NMOS placeholders.
  - connectors.kicad_sch  — 4× SMA for CLK_OUT0–3, 3× SMA for
                            OSC_EN/WEIGHT_EN/SAMPLE_TRIG, 1×4 GPIO
                            header, 3× Keystone-5011 GND test clips.
  - fmc.kicad_sch         — VITA 57.1 LPC connector (4 units × 40 pins),
                            wired for 3P3V/VADJ/SCL/SDA/PRSNT/GA0/GA1/
                            PG_C2M/LDO_EN/LSW_EN; LA-bank pins NC'd for
                            later pinning; all other C/D/G/H pins to GND.

Generator improvements driven by this round:
  - Multi-unit symbol support (parse_pins now returns the per-pin unit
    number; place() takes a unit= parameter and emits matching (unit N)
    in the instance + path).
  - Escape backslash/quote in property values so refs/values with
    embedded " (e.g. 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
Parts:
- added J1, J2, J3, J4, J5, J6, J7: SMA, Connector_Coaxial:SMA_Amphenol_HRM-G_Vertical, symbol Lib:HRM-G-300-467B-1
- added J8: 1x4 100mil, Connector_PinHeader_2.54mm:PinHeader_1x04_P2.54mm_Vertical, symbol Lib:TSW-104-05-G-S
- added TP1, TP2, TP3: GND-CLIP, TestPoint:TestPoint_THTPad_D5.0mm_Drill3.0mm, symbol Lib:Keystone-5011
Connections:
- new net CLK_OUT0: J1.1
- new net CLK_OUT1: J2.1
- new net CLK_OUT2: J3.1
- new net CLK_OUT3: J4.1
- new net GND: TP1.1, TP2.1, TP3.1
- new net GPIO0: J8.1
- new net GPIO1: J8.2
- new net GPIO2: J8.3
- new net GPIO3: J8.4
- new net OSC_EN: J5.1
- new net SAMPLE_TRIG: J7.1
- new net WEIGHT_EN: J6.1

Commit message: Project-wide connectivity audit: refdes uniqueness + hier-label correctness
Added test1/verify_project.py as a kicad-cli-erc substitute (the dev
build doesn't ship _cvpcb.kiface, so sch erc is broken). The verifier
parses all .kicad_sch files and checks:
  1. Duplicate refdes (KiCad's refdes namespace is project-wide).
  2. Parent sheet-pin name + direction matches child hierarchical_label.
  3. Orphan child hierarchical_labels (no matching parent pin).

First run flagged 48 issues. Now reports 0.

Refdes scheme — per-sheet decade ranges so global namespace stays unique:
  FMC 1-9 (J1-J4)
  Power 10-19 (U10/U11, R10/R11, C10-C16, J10-J12)
  Bobcat 20-29 (U20, R20/R21, C20-C25)
  EEPROM 30-39 (U30, R30/R31, C30)
  Bias 40-49 (U40/U41 [U41 dual-unit OPA], Q40-Q43, R40/R41, C40-C43)
  Connectors 50-59 (J50-J57, TP50-TP52)

Hierarchical / global label rework:
  - Parent sheet-pin directions corrected to match child labels (was
    flipped on every Bobcat SPI pin and on FMC's LDO_EN/LSW_EN/LDO_PG).
  - Bobcat SPI labels: passive → input/output as appropriate.
  - Project-wide nets converted to global_label (auto-tie by name, no
    parent pins): SCL, SDA, SAMPLE_OUT*, OSC_EN, WEIGHT_EN, SAMPLE_TRIG,
    BIAS_ISO0/1, CS_L, SCLK, MOSI, MISO, SPI_DMODE, RESET_N.
  - hier_label retained for clean 2-sheet pairs: VADJ, LDO_EN, LDO_PG,
    LSW_EN (FMC ↔ Power); BIAS0/1 (Bias ↔ Bobcat); CLK_OUT0-3, GPIO0-3
    (Bobcat ↔ Connectors).
  - Visual cue in renders: globals render as boxed rectangles; hierarchical
    labels render as arrows — handy when scanning a sheet.

Memory: appended five connectivity-correctness lessons to
feedback_kicad_generator_lessons.md (refdes namespace, parent/child
direction parity, no-passive-for-real-signals, global vs hier decision
table, verify-after-every-change).

Co-Authored-By: Claude Opus 4.7 (1M context) <noreply@anthropic.com>
Parts:
- removed J1, J2, J3, J4, J5, J6, J7: SMA, Connector_Coaxial:SMA_Amphenol_HRM-G_Vertical, symbol Lib:HRM-G-300-467B-1
- removed J8: 1x4 100mil, Connector_PinHeader_2.54mm:PinHeader_1x04_P2.54mm_Vertical, symbol Lib:TSW-104-05-G-S
- removed TP1, TP2, TP3: GND-CLIP, TestPoint:TestPoint_THTPad_D5.0mm_Drill3.0mm, symbol Lib:Keystone-5011
- added J50, J51, J52, J53, J54, J55, J56: SMA, Connector_Coaxial:SMA_Amphenol_HRM-G_Vertical, symbol Lib:HRM-G-300-467B-1
- added J57: 1x4 100mil, Connector_PinHeader_2.54mm:PinHeader_1x04_P2.54mm_Vertical, symbol Lib:TSW-104-05-G-S
- added TP50, TP51, TP52: GND-CLIP, TestPoint:TestPoint_THTPad_D5.0mm_Drill3.0mm, symbol Lib:Keystone-5011
Connections:
- net CLK_OUT0: now also J50.1
- net CLK_OUT1: now also J51.1
- net CLK_OUT2: now also J52.1
- net CLK_OUT3: now also J53.1
- net GND: now also TP50.1, TP51.1, TP52.1
- net GPIO0: now also J57.1
- net GPIO1: now also J57.2
- net GPIO2: now also J57.3
- net GPIO3: now also J57.4
- net OSC_EN: now also J54.1
- net SAMPLE_TRIG: now also J56.1
- net WEIGHT_EN: now also J55.1

Commit message: Split test1 generator into per-sheet package with netlist YAML + strict validator
Combines three layered changes:

1. Apply the design-review audit (test1/error_log.md): 9 ERRORs + 10
   WARNINGs from the new .claude/skills/design_review.md skill — FMC
   LA-bank 0Ω routing, Bobcat SPI/control/GPIO pull network, LDO
   ANY-OUT to FPGA, LDO_PG pull-up + series, bias DNP convention,
   kelvin SNS, per-pin VDDIO + bulk caps, BIAS bypass, VADJ/VDDIO bulk,
   MCP4728 EEPROM provisioning notes, shared-rail decision documented.

2. Refactor test1/gen_schematic.py (1825 lines → 138-line entry point)
   into a per-sheet package at test1/gen/:
     config.py / symbols.py / shared.py  — primitives, Sheet container,
     LA_ASSIGN, footprints, sexpr emit
     build_<sheet>.py × 7                — one builder per child sheet
     netlist.py / validator.py           — YAML loader + strict checker
   Per-session context for any single sheet drops to ~500 lines.
   Also sorts non-deterministic set iteration that made fmc.kicad_sch
   diff noisily across runs.

3. Add a declarative connectivity layer (netlist/<sheet>.yaml):
   parts inventory + nets (power / hier / global / internal), with
   explicit unit syntax for multi-unit symbols (U41:u2.7, J3:u3.G16).
   The strict validator runs at the end of every build_<sheet>() call:
     - inventory: YAML parts ↔ placed (refdes, unit) parity
     - connectivity: every YAML net member is in a connected component
       named the YAML net name (Union-Find on wires + junctions + label
       anchors + power-symbol pins; T-intersections auto-connect)
     - internal nets: members in one component, no name check
   Sheet now records structured PlacedPart/wire/label data alongside
   the s-expr emit; validator reads those instead of re-parsing.

All 6 child sheets' .kicad_sch outputs are byte-identical to the
post-design-review reference, and verify_project.py reports 0 issues.

Co-Authored-By: Claude Opus 4.7 (1M context) <noreply@anthropic.c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
Parts:
- added R50, R51, R52: 0, Resistor_SMD:R_0402_1005Metric, symbol Device:R
Connections:
- net OSC_EN: now also R50.1; no longer J54.1
- net SAMPLE_TRIG: now also R52.1; no longer J56.1
- net WEIGHT_EN: now also R51.1; no longer J55.1
- new net: J55.1, R51.2
- new net: J56.1, R52.2
- new net: J54.1, R50.2
Changed lines of the file:
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@@
       (project "test1"
         (path "/4ed7a046-ef33-57d9-8730-321c05965af3/059bce26-e22e-55b8-805e-999a0610e155" (reference "J54") (unit 1)))))
-  (wire (pts (xy 165 100.0) (xy 157.71 100.0)) (stroke (width 0) (type default)))
-  (global_label "OSC_EN" (shape input) (at 157.71 100.0 180) (effects (font (size 1.27 1.27)) (justify right)))
+  (symbol
+    (lib_id "Device:R")
+    (at 160 100.0 90)
+    (unit 1) (in_bom yes) (on_board yes) (dnp no)
+    (property "Reference" "R50" (at 160 96.19 0) (effects (font (size 1.27 1.27))))
+    (property "Value" "0" (at 160 103.81 0) (effects (font (size 1.27 1.27))))
+    (property "Footprint" "Resistor_SMD:R_0402_1005Metric" (at 0 0 0) (effects (font (size 1.27 1.27)) (hide yes)))
+    (property "Datasheet" "" (at 0 0 0) (effects (font (size 1.27 1.27)) (hide yes)))
+    (pin "1")
+    (pin "2")
+    (instances
+      (project "test1"
+        (path "/4ed7a046-ef33-57d9-8730-321c05965af3/059bce26-e22e-55b8-805e-999a0610e155" (reference "R50") (unit 1)))))
+  (wire (pts (xy 165 100.0) (xy 163.81 100.0)) (stroke (width 0) (type default)))
+  (wire (pts (xy 156.19 100.0) (xy 150 100.0)) (stroke (width 0) (type default)))
+  (global_label "OSC_EN" (shape input) (at 150 100.0 180) (effects (font (size 1.27 1.27)) (justify right)))
   (symbol
     (lib_id "Lib:HRM-G-300-467B-1")
@@
       (project "test1"
         (path "/4ed7a046-ef33-57d9-8730-321c05965af3/059bce26-e22e-55b8-805e-999a0610e155" (reference "J55") (unit 1)))))
-  (wire (pts (xy 165 115.24) (xy 157.71 115.24)) (stroke (width 0) (type default)))
-  (global_label "WEIGHT_EN" (shape input) (at 157.71 115.24 180) (effects (font (size 1.27 1.27)) (justify right)))
+  (symbol
+    (lib_id "Device:R")
+    (at 160 115.24 90)
+    (unit 1) (in_bom yes) (on_board yes) (dnp no)
+    (property "Reference" "R51" (at 160 111.42999999999999 0) (effects (font (size 1.27 1.27))))
+    (property "Value" "0" (at 160 119.05 0) (effects (font (size 1.27 1.27))))
+    (property "Footprint" "Resistor_SMD:R_0402_1005Metric" (at 0 0 0) (effects (font (size 1.27 1.27)) (hide yes)))
+    (property "Datasheet" "" (at 0 0 0) (effects (font (size 1.27 1.27)) (hide yes)))
+    (pin "1")
+    (pin "2")
+    (instances
+      (project "test1"
+        (path "/4ed7a046-ef33-57d9-8730-321c05965af3/059bce26-e22e-55b8-805e-999a0610e155" (reference "R51") (unit 1)))))
+  (wire (pts (xy 165 115.24) (xy 163.81 115.24)) (stroke (width 0) (type default)))
+  (wire (pts (xy 156.19 115.24) (xy 150 115.24)) (stroke (width 0) (type default)))
+  (global_label "WEIGHT_EN" (shape input) (at 150 115.24 180) (effects (font (size 1.27 1.27)) (justify right)))
   (symbol
     (lib_id "Lib:HRM-G-300-467B-1")
@@
       (project "test1"
         (path "/4ed7a046-ef33-57d9-8730-321c05965af3/059bce26-e22e-55b8-805e-999a0610e155" (reference "J56") (unit 1)))))
-  (wire (pts (xy 165 130.48) (xy 157.71 130.48)) (stroke (width 0) (type default)))
-  (global_label "SAMPLE_TRIG" (shape input) (at 157.71 130.48 180) (effects (font (size 1.27 1.27)) (justify right)))
+  (symbol
+    (lib_id "Device:R")
+    (at 160 130.48 90)
+    (unit 1) (in_bom yes) (on_board yes) (dnp no)
+    (property "Reference" "R52" (at 160 126.66999999999999 0) (effects (font (size 1.27 1.27))))
+    (property "Value" "0" (at 160 134.29 0) (effects (font (size 1.27 1.27))))
+    (property "Footprint" "Resistor_SMD:R_0402_1005Metric" (at 0 0 0) (effects (font (size 1.27 1.27)) (hide yes)))
+    (property "Datasheet" "" (at 0 0 0) (effects (font (size 1.27 1.27)) (hide yes)))
+    (pin "1")
+    (pin "2")
+    (instances
+      (project "test1"
+        (path "/4ed7a046-ef33-57d9-8730-321c05965af3/059bce26-e22e-55b8-805e-999a0610e155" (reference "R52") (unit 1)))))
+  (wire (pts (xy 165 130.48) (xy 163.81 130.48)) (stroke (width 0) (type default)))
+  (wire (pts (xy 156.19 130.48) (xy 150 130.48)) (stroke (width 0) (type default)))
+  (global_label "SAMPLE_TRIG" (shape input) (at 150 130.48 180) (effects (font (size 1.27 1.27)) (justify right)))
   (symbol
     (lib_id "Lib:TSW-104-05-G-S")

Commit message: Add layout linter + cluster helpers; fix silent shorts across sheets
Introduces gen/layout_lint.py with checks for bbox spacing, wires
through/into a body, parallel-wire overlap on the same axis, bridged
drop columns, and dense GND clusters — non-fatal warnings the strict
validator cannot catch (each net's name is still present in a bridged
component's name set, so per-member name checks pass).

Fixes the bugs the linter exposed:
- FMC routing flipped to exit LEFT (pin-protrusion side) so wires no
  longer pass through the connector body
- bobcat OWT (pins 23-25) + GPIO (37-40) get one drop column per pin,
  ending the silent shorts between adjacent nets
- bobcat SPI pin 14 pull-x shifted off pin 19's column
- bias Q40/Q41 source/drain wires detoured around the body so source
  no longer shorts to drain through the same vertical
- power LDO redundant tap stubs + GND-rail dupes removed; C12 moved
  off R10's column so NR_SS doesn't short to GND
- C11 ↔ R10, J54-56 ↔ R50-52 spacing widened to meet bbox rule

Adds gnd_bus() and decoupling_cluster() helpers in gen/shared.py and
applies gnd_bus() to the eeprom address-strap pins.

Skill doc gets rules for pin-protrusion side, per-pin drop columns,
and same-axis wire overlap. All 7 sheets now pass kicad-cli parse,
the strict connectivity validator, and the layout linter.

Co-Authored-By: Claude Opus 4.7 (1M context) <noreply@anthropic.com>
Other:
- moved on the sheet: J54, J55, J56
Changed lines of the file:
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@@
   (symbol
     (lib_id "Lib:HRM-G-300-467B-1")
-    (at 165 100.0 0)
+    (at 170 100.0 0)
     (unit 1) (in_bom yes) (on_board yes) (dnp no)
-    (property "Reference" "J54" (at 165 94.92 0) (effects (font (size 1.27 1.27))))
-    (property "Value" "SMA" (at 165 105.08 0) (effects (font (size 1.27 1.27))))
+    (property "Reference" "J54" (at 170 94.92 0) (effects (font (size 1.27 1.27))))
+    (property "Value" "SMA" (at 170 105.08 0) (effects (font (size 1.27 1.27))))
     (property "Footprint" "Connector_Coaxial:SMA_Amphenol_HRM-G_Vertical" (at 0 0 0) (effects (font (size 1.27 1.27)) (hide yes)))
     (property "Datasheet" "" (at 0 0 0) (effects (font (size 1.27 1.27)) (hide yes)))
@@
       (project "test1"
         (path "/4ed7a046-ef33-57d9-8730-321c05965af3/059bce26-e22e-55b8-805e-999a0610e155" (reference "R50") (unit 1)))))
-  (wire (pts (xy 165 100.0) (xy 163.81 100.0)) (stroke (width 0) (type default)))
+  (wire (pts (xy 170 100.0) (xy 163.81 100.0)) (stroke (width 0) (type default)))
   (wire (pts (xy 156.19 100.0) (xy 150 100.0)) (stroke (width 0) (type default)))
   (global_label "OSC_EN" (shape input) (at 150 100.0 180) (effects (font (size 1.27 1.27)) (justify right)))
   (symbol
     (lib_id "Lib:HRM-G-300-467B-1")
-    (at 165 115.24 0)
+    (at 170 115.24 0)
     (unit 1) (in_bom yes) (on_board yes) (dnp no)
-    (property "Reference" "J55" (at 165 110.16 0) (effects (font (size 1.27 1.27))))
-    (property "Value" "SMA" (at 165 120.32 0) (effects (font (size 1.27 1.27))))
+    (property "Reference" "J55" (at 170 110.16 0) (effects (font (size 1.27 1.27))))
+    (property "Value" "SMA" (at 170 120.32 0) (effects (font (size 1.27 1.27))))
     (property "Footprint" "Connector_Coaxial:SMA_Amphenol_HRM-G_Vertical" (at 0 0 0) (effects (font (size 1.27 1.27)) (hide yes)))
     (property "Datasheet" "" (at 0 0 0) (effects (font (size 1.27 1.27)) (hide yes)))
@@
       (project "test1"
         (path "/4ed7a046-ef33-57d9-8730-321c05965af3/059bce26-e22e-55b8-805e-999a0610e155" (reference "R51") (unit 1)))))
-  (wire (pts (xy 165 115.24) (xy 163.81 115.24)) (stroke (width 0) (type default)))
+  (wire (pts (xy 170 115.24) (xy 163.81 115.24)) (stroke (width 0) (type default)))
   (wire (pts (xy 156.19 115.24) (xy 150 115.24)) (stroke (width 0) (type default)))
   (global_label "WEIGHT_EN" (shape input) (at 150 115.24 180) (effects (font (size 1.27 1.27)) (justify right)))
   (symbol
     (lib_id "Lib:HRM-G-300-467B-1")
-    (at 165 130.48 0)
+    (at 170 130.48 0)
     (unit 1) (in_bom yes) (on_board yes) (dnp no)
-    (property "Reference" "J56" (at 165 125.39999999999999 0) (effects (font (size 1.27 1.27))))
-    (property "Value" "SMA" (at 165 135.56 0) (effects (font (size 1.27 1.27))))
+    (property "Reference" "J56" (at 170 125.39999999999999 0) (effects (font (size 1.27 1.27))))
+    (property "Value" "SMA" (at 170 135.56 0) (effects (font (size 1.27 1.27))))
     (property "Footprint" "Connector_Coaxial:SMA_Amphenol_HRM-G_Vertical" (at 0 0 0) (effects (font (size 1.27 1.27)) (hide yes)))
     (property "Datasheet" "" (at 0 0 0) (effects (font (size 1.27 1.27)) (hide yes)))
@@
       (project "test1"
         (path "/4ed7a046-ef33-57d9-8730-321c05965af3/059bce26-e22e-55b8-805e-999a0610e155" (reference "R52") (unit 1)))))
-  (wire (pts (xy 165 130.48) (xy 163.81 130.48)) (stroke (width 0) (type default)))
+  (wire (pts (xy 170 130.48) (xy 163.81 130.48)) (stroke (width 0) (type default)))
   (wire (pts (xy 156.19 130.48) (xy 150 130.48)) (stroke (width 0) (type default)))
   (global_label "SAMPLE_TRIG" (shape input) (at 150 130.48 180) (effects (font (size 1.27 1.27)) (justify right)))
