File: test1/kicad/bias.kicad_sch (KiCad schematic)
At the start: 15 parts, among them Q40 PMZ1200UPEYL, Q41 PMZ1200UPEYL, Q42 2N7002, Q43 2N7002, U40 MCP4728, U41 OPA2388

Commit message: Close W2 by fail-safe redesign: Q42/Q43 populated-default, FPGA-gated bias
Previously the bias circuit was fail-deadly: a virgin MCP4728 (factory
default VREF=2.048V, code=0x000) would drive V_DAC=0V → PMOS fully on
→ ~646 µA into Bobcat the instant +3.3V came up, before any I²C
intervention. The only thing protecting the DUT was somebody
remembering an assembly-time provisioning step.

The design already shipped the hardware hooks for a fail-safe
isolation path — Q42/Q43 (2N7002 NMOSes) in series between PMOS drain
and BIAS pins, with R44/R45 10kΩ pull-downs holding their gates LOW
at POR. They were just DNP, with R42/R43 0Ω jumpers populated as the
permanent override.

This commit flips the convention:
  netlist/bias.yaml:
    Q42, Q43          → populated-default (dnp removed)
    R42, R43          → DNP-default (dnp: true)
    notes refreshed to spell out the fail-safe intent

  gen/shared.py:
    + text()          → emits free-form `(text …)` annotations
                        for design-intent notes (doesn't form nets)

  gen/build_bias.py:
    + sheet-level banner near (80, 60) — 7 lines documenting the
      POR fail-safe story
    + per-channel notes below each BIAS_ISO pull-down cluster
      so a future reader doesn't repopulate R42/R43 without
      understanding what they're disabling

  design_requirements.md:
    Bias circuit bullet rewritten to describe the new default
    Assembly note W8 rewritten — provisioning is now recoverable,
      not DUT-fatal (DAC is hardware-isolated until FPGA enables)
    Assembly note for Q42/Q43 (E7) rewritten — reflects new default

Result:
  - W2 hazard mitigated at schematic level. Verified by an
    independent semantic-review agent dispatched after the change.
  - Pipeline state: 0 ERRORs, 0 WARNINGs, 0 INFOs.
  - Build still clean: 0 ERROR, 17 WARNING, 12 INFO (no new findings).

Failure modes the new design handles safely (was → is):
  Tech forgets to program EEPROM:      DUT damaged → DUT safe
  MCP4728 EEPRO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
Parts:
- Q42, Q43: now fitted
- R42, R43: now not fitted
Other:
- note added: "(gate pull-downs R44/R45). FPGA must assert BIAS_ISO0/1 HIGH to"
- note added: "BIAS BLOCK — POR FAIL-SAFE"
- note added: "FAIL-SAFE: BIAS_ISO0 default-LOW (R44 pull-down)"
- note added: "FAIL-SAFE: BIAS_ISO1 default-LOW (R45 pull-down)"
- note added: "Q42/Q43 isolation NMOSes are POPULATED by default and DEFAULT-OFF"
- note added: "R42 is DNP — populate ONLY to bypass FPGA control."
- note added: "R42/R43 (parallel 0Ω) are DNP — populate ONLY to disable the FPGA"
- note added: "R43 is DNP — populate ONLY to bypass FPGA control."
- note added: "code=0x000) cannot push uncontrolled current at POR."
- note added: "deliver bias to Bobcat — a virgin MCP4728 (default VREF=2.048V,"
- note added: "isolation path (benchtop standalone use without FPGA control)."
- note added: "→ Q42 OFF at POR → no bias to Bobcat until FPGA asserts HIGH."
- note added: "→ Q43 OFF at POR → no bias to Bobcat until FPGA asserts HIGH."
Changed lines of the file:
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@@
     (rev "1")
   )
+  (text "BIAS BLOCK — POR FAIL-SAFE" (at 80.0 60.0 0) (effects (font (size 1.5 1.5)) (justify left)))
+  (text "Q42/Q43 isolation NMOSes are POPULATED by default and DEFAULT-OFF" (at 80.0 63.0 0) (effects (font (size 0.9 0.9)) (justify left)))
+  (text "(gate pull-downs R44/R45). FPGA must assert BIAS_ISO0/1 HIGH to" (at 80.0 64.5 0) (effects (font (size 0.9 0.9)) (justify left)))
+  (text "deliver bias to Bobcat — a virgin MCP4728 (default VREF=2.048V," (at 80.0 66.0 0) (effects (font (size 0.9 0.9)) (justify left)))
+  (text "code=0x000) cannot push uncontrolled current at POR." (at 80.0 67.5 0) (effects (font (size 0.9 0.9)) (justify left)))
+  (text "R42/R43 (parallel 0Ω) are DNP — populate ONLY to disable the FPGA" (at 80.0 69.5 0) (effects (font (size 0.9 0.9)) (justify left)))
+  (text "isolation path (benchtop standalone use without FPGA control)." (at 80.0 71.0 0) (effects (font (size 0.9 0.9)) (justify left)))
   (symbol
     (lib_id "Lib:MCP4728")
@@
     (lib_id "Lib:2N7002")
     (at 250.0 115.08 0)
-    (unit 1) (in_bom yes) (on_board yes) (dnp yes)
+    (unit 1) (in_bom yes) (on_board yes) (dnp no)
     (property "Reference" "Q42" (at 250.0 110.0 0) (effects (font (size 1.27 1.27))))
     (property "Value" "2N7002" (at 250.0 120.16 0) (effects (font (size 1.27 1.27))))
@@
     (lib_id "Device:R")
     (at 265.24 115.08 0)
-    (unit 1) (in_bom yes) (on_board yes) (dnp no)
+    (unit 1) (in_bom yes) (on_board yes) (dnp yes)
     (property "Reference" "R42" (at 267.78 113.81 0) (effects (font (size 1.27 1.27))))
     (property "Value" "0" (at 267.78 116.35 0) (effects (font (size 1.27 1.27))))
@@
       (project "test1"
         (path "/4ed7a046-ef33-57d9-8730-321c05965af3/ddf1c49f-55ac-530a-9ee4-38ad9d14caf8" (reference "#PWRe0ee7a24") (unit 1)))))
+  (text "FAIL-SAFE: BIAS_ISO0 default-LOW (R44 pull-down)" (at 239.84 132.86 0) (effects (font (size 0.8 0.8)) (justify left)))
+  (text "→ Q42 OFF at POR → no bias to Bobcat until FPGA asserts HIGH." (at 239.84 134.36 0) (effects (font (size 0.8 0.8)) (justify left)))
+  (text "R42 is DNP — populate ONLY to bypass FPGA control." (at 239.84 135.86 0) (effects (font (size 0.8 0.8)) (justify left)))
   (wire (pts (xy 215.16 104.92) (xy 215.16 99.84)) (stroke (width 0) (type default)))
   (symbol
@@
     (lib_id "Lib:2N7002")
     (at 365.0 115.08 0)
-    (unit 1) (in_bom yes) (on_board yes) (dnp yes)
+    (unit 1) (in_bom yes) (on_board yes) (dnp no)
     (property "Reference" "Q43" (at 365.0 110.0 0) (effects (font (size 1.27 1.27))))
     (property "Value" "2N7002" (at 365.0 120.16 0) (effects (font (size 1.27 1.27))))
@@
     (lib_id "Device:R")
     (at 380.24 115.08 0)
-    (unit 1) (in_bom yes) (on_board yes) (dnp no)
+    (unit 1) (in_bom yes) (on_board yes) (dnp yes)
     (property "Reference" "R43" (at 382.78 113.81 0) (effects (font (size 1.27 1.27))))
     (property "Value" "0" (at 382.78 116.35 0) (effects (font (size 1.27 1.27))))
@@
       (project "test1"
         (path "/4ed7a046-ef33-57d9-8730-321c05965af3/ddf1c49f-55ac-530a-9ee4-38ad9d14caf8" (reference "#PWRad49c2e3") (unit 1)))))
+  (text "FAIL-SAFE: BIAS_ISO1 default-LOW (R45 pull-down)" (at 354.84 132.86 0) (effects (font (size 0.8 0.8)) (justify left)))
+  (text "→ Q43 OFF at POR → no bias to Bobcat until FPGA asserts HIGH." (at 354.84 134.36 0) (effects (font (size 0.8 0.8)) (justify left)))
+  (text "R43 is DNP — populate ONLY to bypass FPGA control." (at 354.84 135.86 0) (effects (font (size 0.8 0.8)) (justify left)))
   (symbol
     (lib_id "Device:C")
