File: test1/kicad/bias.kicad_sch (KiCad schematic)
At the start: 15 parts, among them Q40 PMZ1200UPEYL, Q41 PMZ1200UPEYL, Q42 2N7002, Q43 2N7002, U40 MCP4728, U41 OPA2388

Commit message: Add AI-assisted simulation subsystem with context-first pipeline
Catalog-driven ngspice sim layer (test1/sim): per-block decks for LDO
rail, OPA bias loop, and PDN, with boundary stubs, datasheet-grounded
param mapping, bounded re-sim iteration, and fault-injection self-tests.
Wires a Simulation tab into the GUI: datasheet-tagged blocks, workflow
status steps, agent thinking checklist, and checkable circuit-edit
suggestions that push to the changelog.

Co-Authored-By: Claude Opus 4.7 <noreply@anthropic.com>
Other:
- note added: "FPGA must drive BIAS_ISO0/1 HIGH; MCP4728 defaults (VREF=2.048V, code=0) are safe."
- note added: "Q42/Q43 (populated, default-OFF via R44/R45) block bias at POR."
- note added: "R42/R43 DNP — short only for FPGA-less benchtop use."
- note removed: "(gate pull-downs R44/R45). FPGA must assert BIAS_ISO0/1 HIGH to"
- note removed: "Q42/Q43 isolation NMOSes are POPULATED by default and DEFAULT-OFF"
- note removed: "R42/R43 (parallel 0Ω) are DNP — populate ONLY to disable the FPGA"
- note removed: "code=0x000) cannot push uncontrolled current at POR."
- note removed: "deliver bias to Bobcat — a virgin MCP4728 (default VREF=2.048V,"
- note removed: "isolation path (benchtop standalone use without FPGA control)."
Changed lines of the file:
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@@
   )
   (text "BIAS BLOCK — POR FAIL-SAFE" (at 80.0 60.0 0) (effects (font (size 1.5 1.5)) (justify left)))
-  (text "Q42/Q43 isolation NMOSes are POPULATED by default and DEFAULT-OFF" (at 80.0 63.0 0) (effects (font (size 0.9 0.9)) (justify left)))
-  (text "(gate pull-downs R44/R45). FPGA must assert BIAS_ISO0/1 HIGH to" (at 80.0 64.5 0) (effects (font (size 0.9 0.9)) (justify left)))
-  (text "deliver bias to Bobcat — a virgin MCP4728 (default VREF=2.048V," (at 80.0 66.0 0) (effects (font (size 0.9 0.9)) (justify left)))
-  (text "code=0x000) cannot push uncontrolled current at POR." (at 80.0 67.5 0) (effects (font (size 0.9 0.9)) (justify left)))
-  (text "R42/R43 (parallel 0Ω) are DNP — populate ONLY to disable the FPGA" (at 80.0 69.5 0) (effects (font (size 0.9 0.9)) (justify left)))
-  (text "isolation path (benchtop standalone use without FPGA control)." (at 80.0 71.0 0) (effects (font (size 0.9 0.9)) (justify left)))
+  (text "Q42/Q43 (populated, default-OFF via R44/R45) block bias at POR." (at 80.0 63.0 0) (effects (font (size 0.9 0.9)) (justify left)))
+  (text "FPGA must drive BIAS_ISO0/1 HIGH; MCP4728 defaults (VREF=2.048V, code=0) are safe." (at 80.0 65.0 0) (effects (font (size 0.9 0.9)) (justify left)))
+  (text "R42/R43 DNP — short only for FPGA-less benchtop use." (at 80.0 67.0 0) (effects (font (size 0.9 0.9)) (justify left)))
   (symbol
     (lib_id "Lib:MCP4728")
