File: test1/kicad/bobcat.kicad_sch (KiCad schematic)
At the start: 25 parts, among them U20 Bobcat

Commit message: Add AI-assisted simulation subsystem with context-first pipeline
Catalog-driven ngspice sim layer (test1/sim): per-block decks for LDO
rail, OPA bias loop, and PDN, with boundary stubs, datasheet-grounded
param mapping, bounded re-sim iteration, and fault-injection self-tests.
Wires a Simulation tab into the GUI: datasheet-tagged blocks, workflow
status steps, agent thinking checklist, and checkable circuit-edit
suggestions that push to the changelog.

Co-Authored-By: Claude Opus 4.7 <noreply@anthropic.com>
Other:
- note added: "VDDD core bypass"
- note added: "VDDIO supply bypass"
Changed lines of the file:
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@@
       (project "test1"
         (path "/4ed7a046-ef33-57d9-8730-321c05965af3/e6b90fa2-2dfc-5319-a99a-2ebf8a1933a0" (reference "#PWR73ac9cc2") (unit 1)))))
+  (text "VDDD core bypass" (at 187.96 167.64 0) (effects (font (size 1.0 1.0)) (justify right)))
   (symbol
     (lib_id "Device:R")
@@
       (project "test1"
         (path "/4ed7a046-ef33-57d9-8730-321c05965af3/e6b90fa2-2dfc-5319-a99a-2ebf8a1933a0" (reference "#PWR2794fcca") (unit 1)))))
+  (text "VDDIO supply bypass" (at 137.16 100.33 0) (effects (font (size 1.0 1.0)) (justify right)))
   (wire (pts (xy 195.58 152.4) (xy 195.58 185.42)) (stroke (width 0) (type default)))
   (wire (pts (xy 195.58 185.42) (xy 165.1 185.42)) (stroke (width 0) (type default)))
