File: test1/kicad/power.kicad_sch (KiCad schematic)
At the start: 17 parts, among them J10 1x2 100mil, J11 1x2 100mil, J12 1x2 100mil, U10 TPS7A8401A, U11 TPS22916

Commit message: Add AI-assisted simulation subsystem with context-first pipeline
Catalog-driven ngspice sim layer (test1/sim): per-block decks for LDO
rail, OPA bias loop, and PDN, with boundary stubs, datasheet-grounded
param mapping, bounded re-sim iteration, and fault-injection self-tests.
Wires a Simulation tab into the GUI: datasheet-tagged blocks, workflow
status steps, agent thinking checklist, and checkable circuit-edit
suggestions that push to the changelog.

Co-Authored-By: Claude Opus 4.7 <noreply@anthropic.com>
Other:
- note added: "LDO VIN bypass"
- note added: "LDO VOUT bypass"
Changed lines of the file:
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@@
       (project "test1"
         (path "/4ed7a046-ef33-57d9-8730-321c05965af3/45af8917-b3aa-56de-8c9b-8d649d910e5f" (reference "#PWR091e800f") (unit 1)))))
+  (text "LDO VIN bypass" (at 80.01 129.54 0) (effects (font (size 1.0 1.0)) (justify right)))
   (wire (pts (xy 109.22 119.38) (xy 99.06 119.38)) (stroke (width 0) (type default)))
   (symbol
@@
   (wire (pts (xy 180.34 125.73) (xy 180.34 119.38)) (stroke (width 0) (type default)))
   (wire (pts (xy 180.34 133.35) (xy 180.34 175.26)) (stroke (width 0) (type default)))
+  (text "LDO VOUT bypass" (at 170.18 129.54 0) (effects (font (size 1.0 1.0)) (justify right)))
   (symbol
     (lib_id "Lib:TSW-102-05-G-S")
