File: test1/kicad/test1.kicad_sch (KiCad schematic)
At the start: 0 parts

Commit message: Migrate symbols to Ultra Librarian parts; add Altium pipeline + GUI/BOM updates
Library:
- Replace per-MPN symbols with Ultra Librarian .SchLib + .PcbLib (16 parts);
  swap bulk MLCC CC0805KFX7R6BB106 -> GRM21BR71A106KA73L; drop legacy .kicad_sym.
- 2N7002 kept on the original MOSFET symbol (the UL download was a SOT-23 diode).

build_symbols: rebuild merged parts.SchLib when a source symbol is newer
(mtime), and resolve each symbol's real internal name instead of assuming the
MPN (UL names differ, e.g. OPA2388 -> OPA2388IDGKR).

Sheets re-routed for the new UL pin maps (builders wire to real pin coords):
- bias: single-unit OPA2388 (U41 placed once, both channels routed to it;
  netlist collapsed to one unit) + MCP4728 (U40) new pin layout.
- power: TPS7A8401A (U10) input/setpoint/output regrouped; TSW-102 jumper
  centering. fmc: stagger +3V3/GND power-symbol columns.
All six sheets build 0 errors / 0 warnings.

Build: layout auto-fix pass nudges cosmetic note overlaps clear
(shared.auto_fix_text), run per sheet by build_project.

GUI: per-part .SchLib upload + Ultra Librarian deep link in the Library tab;
fix Generate (apply-and-generate) to drive the Altium backend instead of the
KiCad gen_schematic.py.

BOM: point C_bulk at GRM21BR71A106KA73L; drop unused columns (Manufacturer,
Distributor, Distributor P/N, Unit Price); sync generate_bom.py.

Docs: add docs/pipeline.tex describing the workflow/pipeline.

Co-Authored-By: Claude Opus 4.7 (1M context) <noreply@anthropic.com>
Other:
- title: test1 — Bobcat Carrier (root) -> test1  Bobcat Carrier (root)
Changed lines of the file:
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@@
   (paper "A3")
   (title_block
-    (title "test1 — Bobcat Carrier (root)")
+    (title "test1  Bobcat Carrier (root)")
     (date "")
     (rev "1")
